File: rfid.kicad_sch (KiCad schematic)
At the start: 37 parts, among them U1 ATtiny25-20SS

Commit message: New version
Parts:
- SW1: footprint X7:PowerSwitch -> X7:CL-SB-12A-11T
Changed lines of the file:
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@@
 			)
 		)
-		(property "Footprint" "X7:PowerSwitch"
+		(property "Footprint" "X7:CL-SB-12A-11T"
 			(at 71.12 99.06 0)
 			(effects
@@
 					(size 1.27 1.27)
 				)
-				(hide yes)
 			)
 		)

Commit message: FInal
Parts:
- added BUZZER1, DEMOD1, GND1, TP1_R, TP2_D: TestPoint, TestPoint:TestPoint_THTPad_D2.0mm_Drill1.0mm, symbol Connector:TestPoint
- L1: footprint (none) -> Passives:COIL
Connections:
- net BUZZER: now also BUZZER1.1
- net DEMOD: now also DEMOD1.1
- net GND: now also GND1.1
- net at C1.1, C1A1.1, D1.2 (A)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: now also TP2_D.1
- net at L1.1, R1.1: now also TP1_R.1
